Commit message: added scene cameras to the xacro

File: clr_description/urdf/clr_macro.xacro (robot description, xacro)
@@ -184,4 +184,22 @@
       <origin xyz="-0.0772 0.095 0.2635" rpy="0 0 0"/>
     </xacro:lift_camera>
+    <!-- Left and Right Scene Cameras -->
+    <xacro:include filename="$(find clr_description)/urdf/scene_camera.macro.xacro"/>
+    <xacro:scene_camera
+      tf_prefix="${tf_prefix}"
+      parent="world"
+      name="left_scene_camera"
+      use_camera_mesh="${use_camera_mesh}"
+    >
+      <origin xyz="-0.6 1.0 2.2" rpy="0 0 0"/>
+    </xacro:scene_camera>
+    <xacro:scene_camera
+      tf_prefix="${tf_prefix}"
+      name="right_scene_camera"
+      parent="world"
+      use_camera_mesh="${use_camera_mesh}"
+    >
+      <origin xyz="0.51 1.17 2.2" rpy="0 0 0"/>
+    </xacro:scene_camera>
     <!-- UPPER_LIFT_PLATE -->
     <xacro:upper_lift_plate

Commit message: these cmaeras......

File: clr_description/urdf/clr_macro.xacro (robot description, xacro)
@@ -192,5 +192,9 @@
       use_camera_mesh="${use_camera_mesh}"
     >
-      <origin xyz="-0.6 1.0 2.2" rpy="0 0 0"/>
+      <!-- <origin xyz="-0.372 1.284 2.596" rpy="0.933 -0.345 -0.101"/> -->
+      <!-- <origin xyz="-0.372 1.284 2.596" rpy="1.952  0.265 -0.105"/> -->
+      <!-- <origin xyz="-0.372 1.284 2.596" rpy="0.285 -0.000  1.938"/> -->
+      <!-- <origin xyz="-0.372 1.284 2.596" rpy="-0.105246 0.2648029 1.9527127"/> -->
+      <origin xyz="-0.372 1.284 2.596" rpy="1.570 1.286 -2.775"/>
     </xacro:scene_camera>
     <xacro:scene_camera
@@ -200,5 +204,10 @@
       use_camera_mesh="${use_camera_mesh}"
     >
-      <origin xyz="0.51 1.17 2.2" rpy="0 0 0"/>
+      <!-- <origin xyz="-1.482 1.114 2.596" rpy="-1.594 -0.348 -0.008"/> -->
+      <!-- <origin xyz="-1.482 1.114 2.596" rpy="0.348  0.000 -1.593"/> -->
+      <!-- xyz -->
+      <!-- <origin xyz="-1.482 1.114 2.596" rpy="-0.0083523 -0.3481073 -1.5938004"/> -->
+      <!-- zyx -->
+      <origin xyz="-1.482 1.114 2.596" rpy="1.567 1.223 -0.025"/>
     </xacro:scene_camera>
     <!-- UPPER_LIFT_PLATE -->

File: clr_description/urdf/scene_camera.macro.xacro (robot description, xacro)
@@ -18,7 +18,9 @@
     <link name="${tf_prefix}${name}_mount">
         <visual>
-            <origin rpy="0 0 0" xyz="${mount_width_meters/2} ${-1*mount_depth_meters/2} ${-1*mount_height_meters/2}"/>
+            <!-- <origin rpy="0 0 0" xyz="${mount_width_meters/2} ${-1*mount_depth_meters/2} ${-1*mount_height_meters/2}"/> -->
+            <origin rpy="0 0 0" xyz="0 0 0"/>
             <geometry>
-                <box size="${mount_width_meters} ${mount_depth_meters} ${mount_height_meters}"/> <!--meters -->
+                <!-- <box size="${mount_width_meters} ${mount_depth_meters} ${mount_height_meters}"/> meters -->
+                <box size="0.01 0.01 0.01"/> <!--meters -->
             </geometry>
             <material name="${tf_prefix}${name}_mount">
@@ -27,7 +29,9 @@
         </visual>
         <collision>
-            <origin rpy="0 0 0" xyz="${mount_width_meters/2} ${-1*mount_depth_meters/2} ${-1*mount_height_meters/2}"/>
+            <!-- <origin rpy="0 0 0" xyz="${mount_width_meters/2} ${-1*mount_depth_meters/2} ${-1*mount_height_meters/2}"/> -->
+            <origin rpy="0 0 0" xyz="0 0 0"/>
             <geometry>
-                <box size="${mount_width_meters} ${mount_depth_meters} ${mount_height_meters}"/> <!--meters -->
+                <!-- <box size="${mount_width_meters} ${mount_depth_meters} ${mount_height_meters}"/> meters -->
+                <box size="0.01 0.01 0.01"/> <!--meters -->
             </geometry>
         </collision>
@@ -48,4 +52,5 @@
     <xacro:sensor_d435 parent="${tf_prefix}${name}_mount" use_nominal_extrinsics="true" use_mesh="${use_camera_mesh}" name="${name}">
         <!-- <origin xyz="-0.007666 0.1069 0.3866" rpy="-3.0512 -0.0276 1.5884"/> -->
+        <origin xyz="0.0 0.0 0.0" rpy="0.0 0.0 0.0"/>
     </xacro:sensor_d435>
     </xacro:macro>

Commit message: fixed transforms

File: clr_description/urdf/clr_macro.xacro (robot description, xacro)
@@ -192,9 +192,6 @@
       use_camera_mesh="${use_camera_mesh}"
     >
-      <!-- <origin xyz="-0.372 1.284 2.596" rpy="0.933 -0.345 -0.101"/> -->
-      <!-- <origin xyz="-0.372 1.284 2.596" rpy="1.952  0.265 -0.105"/> -->
-      <!-- <origin xyz="-0.372 1.284 2.596" rpy="0.285 -0.000  1.938"/> -->
-      <!-- <origin xyz="-0.372 1.284 2.596" rpy="-0.105246 0.2648029 1.9527127"/> -->
-      <origin xyz="-0.372 1.284 2.596" rpy="1.570 1.286 -2.775"/>
+    <!-- Values calculated based on Giovanni's camera placement in the scene -->
+      <origin xyz="-1.498697 1.0813555220000002 2.601912082" rpy="0.00015992907444591954 1.2228742441799936 -0.021996451697037067" />
     </xacro:scene_camera>
     <xacro:scene_camera
@@ -204,10 +201,6 @@
       use_camera_mesh="${use_camera_mesh}"
     >
-      <!-- <origin xyz="-1.482 1.114 2.596" rpy="-1.594 -0.348 -0.008"/> -->
-      <!-- <origin xyz="-1.482 1.114 2.596" rpy="0.348  0.000 -1.593"/> -->
-      <!-- xyz -->
-      <!-- <origin xyz="-1.482 1.114 2.596" rpy="-0.0083523 -0.3481073 -1.5938004"/> -->
-      <!-- zyx -->
-      <origin xyz="-1.482 1.114 2.596" rpy="1.567 1.223 -0.025"/>
+    <!-- Values calculated based on Giovanni's camera placement in the scene -->
+      <origin xyz="-0.369328097 1.320383669 2.60289479" rpy="-0.0002902088964777949 1.2858154441839171 -2.7742751828866092" />
     </xacro:scene_camera>
     <!-- UPPER_LIFT_PLATE -->

File: clr_description/urdf/scene_camera.macro.xacro (robot description, xacro)
@@ -51,5 +51,4 @@
     <xacro:include filename="$(find realsense2_description)/urdf/_d435.urdf.xacro" />
     <xacro:sensor_d435 parent="${tf_prefix}${name}_mount" use_nominal_extrinsics="true" use_mesh="${use_camera_mesh}" name="${name}">
-        <!-- <origin xyz="-0.007666 0.1069 0.3866" rpy="-3.0512 -0.0276 1.5884"/> -->
         <origin xyz="0.0 0.0 0.0" rpy="0.0 0.0 0.0"/>
     </xacro:sensor_d435>
