Commit message: added group state

File: clr_moveit_config/srdf/clr_macro.srdf.xacro (robot description, xacro)
@@ -89,4 +89,12 @@
         <joint name="wrist_2_joint" value="-1.468212906514303" />
         <joint name="wrist_3_joint" value="0.03171319141983986" />
+      </group_state>
+      <group_state name="bag_pick_up" group="ur_manipulator">
+        <joint name="elbow_joint" value="-2.089" />
+        <joint name="shoulder_lift_joint" value="0.238" />
+        <joint name="shoulder_pan_joint" value="1.189" />
+        <joint name="wrist_1_joint" value="-0.985" />
+        <joint name="wrist_2_joint" value="1.936" />
+        <joint name="wrist_3_joint" value="3.14159" />
       </group_state>
       <end_effector group="hand" name="hand" parent_group="ur_manipulator" parent_link="tool0"/>

Commit message: updated initial joint states, and group for the srdf

File: clr_moveit_config/srdf/clr_macro.srdf.xacro (robot description, xacro)
@@ -47,4 +47,12 @@
         <joint name="${tf_prefix}finger_1_joint" value="0"/>
         <joint name="${tf_prefix}finger_2_joint" value="0"/>
+      </group_state>
+      <group_state name="vla_home" group="ur_manipulator">
+        <joint name="${tf_prefix}elbow_joint" value="-2.089" />
+        <joint name="${tf_prefix}shoulder_lift_joint" value="0.238" />
+        <joint name="${tf_prefix}shoulder_pan_joint" value="1.189" />
+        <joint name="${tf_prefix}wrist_1_joint" value="-0.985" />
+        <joint name="${tf_prefix}wrist_2_joint" value="1.936" />
+        <joint name="${tf_prefix}wrist_3_joint" value="3.14159" />
       </group_state>
       <group_state name="home" group="ur_manipulator">

File: clr_mujoco_config/urdf/clr_mujoco_ros2_control_macros.xacro (robot description, xacro)
@@ -53,5 +53,5 @@
       <command_interface name="position"/>
       <state_interface name="position">
-        <param name="initial_value">${3.1927}</param>
+        <param name="initial_value">${1.189}</param>
       </state_interface>
       <state_interface name="velocity"/>
@@ -61,5 +61,5 @@
       <command_interface name="position"/>
       <state_interface name="position">
-        <param name="initial_value">${-2.3913}</param>
+        <param name="initial_value">${0.238}</param>
       </state_interface>
       <state_interface name="velocity"/>
@@ -69,5 +69,5 @@
       <command_interface name="position"/>
       <state_interface name="position">
-        <param name="initial_value">${-1.7760}</param>
+        <param name="initial_value">${-2.089}</param>
       </state_interface>
       <state_interface name="velocity"/>
@@ -77,5 +77,5 @@
       <command_interface name="position"/>
       <state_interface name="position">
-        <param name="initial_value">${-0.4700}</param>
+        <param name="initial_value">${-0.985}</param>
       </state_interface>
       <state_interface name="velocity"/>
@@ -85,5 +85,5 @@
       <command_interface name="position"/>
       <state_interface name="position">
-        <param name="initial_value">${-1.6177}</param>
+        <param name="initial_value">${1.936}</param>
       </state_interface>
       <state_interface name="velocity"/>
@@ -93,5 +93,5 @@
       <command_interface name="position"/>
       <state_interface name="position">
-        <param name="initial_value">${-1.6177}</param>
+        <param name="initial_value">${3.14159}</param>
       </state_interface>
       <state_interface name="velocity"/>
